Commit message: 重装保存

File: legged_gym/resources/robots/02_encos/Serial/urdf/CASBOT02_ENCOS_5dof_skeleton_20250904.urdf (robot description, URDF)
Before this commit: robot CB02_URDF(ECS-WK)0904B, 35 links, 34 joints
Links:
- added link left_hand_link, mass 0.015733; collision mesh filename=../meshes/left_hand_link.STL; visual mesh filename=../meshes/left_hand_link.STL
- added link right_hand_link, mass 0.01573344; collision mesh filename=../meshes/right_hand_link.STL; visual mesh filename=../meshes/right_hand_link.STL
Joints:
- added joint left_hand_joint: type revolute, parent left_wrist_yaw_link, child left_hand_link, origin xyz=0 0 -0.1004 rpy=0 0 0, axis 0 0 1, limit lower=0 upper=0 effort=0 velocity=0
- added joint right_hand_joint: type revolute, parent right_wrist_yaw_link, child right_hand_link, origin xyz=0 -0.00040261 -0.1034 rpy=0 0 0, axis 0 0 1, limit lower=0 upper=0 effort=0 velocity=0
- joint left_shoulder_roll_joint: limit lower=-0.3491 upper=1.5716 effort=75 velocity=12.2 -> lower=-0.0 upper=1.5716 effort=75 velocity=12.2
- joint right_shoulder_roll_joint: limit lower=-1.5716 upper=0.3491 effort=75 velocity=12.2 -> lower=-1.5716 upper=0.0 effort=75 velocity=12.2

File: legged_gym/resources/robots/CAS02/urdf/CB02_URDF(ECS-WK)-1.urdf (robot description, URDF)
Before this commit: robot CASBOT_02, 35 links, 34 joints
Links:
- removed link auxiliary_left_leg_ankle_roll_link1
- removed link auxiliary_left_leg_ankle_roll_link2
- removed link auxiliary_left_leg_ankle_roll_link3
- removed link auxiliary_left_leg_ankle_roll_link4
- removed link auxiliary_right_leg_ankle_roll_link1
- removed link auxiliary_right_leg_ankle_roll_link2
- removed link auxiliary_right_leg_ankle_roll_link3
- removed link auxiliary_right_leg_ankle_roll_link4
- removed link keyframe_head_link
- added link left_hand_link, mass 0.086038; collision mesh filename=../meshes/left_hand_link.STL; visual mesh filename=../meshes/left_hand_link.STL
- added link right_hand_link, mass 0.086038; collision mesh filename=../meshes/right_hand_link.STL; visual mesh filename=../meshes/right_hand_link.STL
- link base_link: mass 4.4711 -> 1.28818193551437; geometry visual mesh filename=../meshes/base_link.STL
- link head_pitch_link: mass 0.095791 -> 0.473264225353606; geometry collision sphere radius=0.07; visual mesh filename=../meshes/head_pitch_link.STL
- link head_yaw_link: mass 0.46029 -> 0.0797810246710037; geometry visual mesh filename=../meshes/head_yaw_link.STL
- link left_elbow_pitch_link: mass 1.6315 -> 0.435303751733877; geometry collision mesh filename=../meshes/left_elbow_pitch_link.STL; visual mesh filename=../meshes/left_elbow_pitch_link.STL
- link left_leg_ankle_pitch_link: mass 0.084483 -> 0.0573757039077953; geometry visual mesh filename=../meshes/left_leg_ankle_pitch_link.STL
- link left_leg_ankle_roll_link: mass 0.63694 -> 0.84968; geometry collision box size=0.23 0.08 0.02; visual mesh filename=../meshes/left_leg_ankle_roll_link.STL
- link left_leg_knee_pitch_link: mass 3.785 -> 3.70179178417344; geometry collision box size=0.03 0.06 0.1; collision box size=0.05 0.07 0.19
- link left_leg_pelvic_pitch_link: mass 2.1606 -> 1.02810145292751; geometry collision cylinder length=0.08 radius=0.06; visual mesh filename=../meshes/left_leg_pelvic_pitch_link.STL
- link left_leg_pelvic_roll_link: mass 0.53073 -> 0.463419741183663; geometry visual mesh filename=../meshes/left_leg_pelvic_roll_link.STL
- link left_leg_pelvic_yaw_link: mass 3.7187 -> 3.92267293403735; geometry visual mesh filename=../meshes/left_leg_pelvic_yaw_link.STL
- link left_shoulder_pitch_link: mass 1.0755 -> 0.649287739116578; geometry visual mesh filename=../meshes/left_shoulder_pitch_link.STL
- link left_shoulder_roll_link: mass 0.6379 -> 0.195328921491811; geometry collision mesh filename=../meshes/left_shoulder_roll_link.STL; visual mesh filename=../meshes/left_shoulder_roll_link.STL
- link left_shoulder_yaw_link: mass 0.087762 -> 0.0243504547014443; geometry collision mesh filename=../meshes/left_shoulder_yaw_link.STL; visual mesh filename=../meshes/left_shoulder_yaw_link.STL
- link left_wrist_yaw_link: mass 0.44922 -> 0.124402127918901; geometry collision mesh filename=../meshes/left_wrist_yaw_link.STL; visual mesh filename=../meshes/left_wrist_yaw_link.STL
- link right_elbow_pitch_link: mass 1.6833 -> 0.435399198132512; geometry collision mesh filename=../meshes/right_elbow_pitch_link.STL; visual mesh filename=../meshes/right_elbow_pitch_link.STL
- link right_leg_ankle_pitch_link: mass 0.084483 -> 0.0573757039077936; geometry visual mesh filename=../meshes/right_leg_ankle_pitch_link.STL
- link right_leg_ankle_roll_link: mass 0.63694 -> 0.84963; geometry collision box size=0.23 0.08 0.02; visual mesh filename=../meshes/right_leg_ankle_roll_link.STL
- link right_leg_knee_pitch_link: mass 3.7883 -> 1.24759478576868; geometry collision box size=0.03 0.06 0.1; collision box size=0.05 0.07 0.19
- link right_leg_pelvic_pitch_link: mass 2.1733 -> 1.71831066939471; geometry collision cylinder length=0.08 radius=0.06; visual mesh filename=../meshes/right_leg_pelvic_pitch_link.STL
- link right_leg_pelvic_roll_link: mass 0.53073 -> 0.463419741183666; geometry visual mesh filename=../meshes/right_leg_pelvic_roll_link.STL
- link right_leg_pelvic_yaw_link: mass 3.7181 -> 4.00564660690577; geometry visual mesh filename=../meshes/right_leg_pelvic_yaw_link.STL
- link right_shoulder_pitch_link: mass 1.0872 -> 0.15551625340884; geometry visual mesh filename=../meshes/right_shoulder_pitch_link.STL
- link right_shoulder_roll_link: mass 0.64426 -> 0.195463682958999; geometry collision mesh filename=../meshes/right_shoulder_roll_link.STL; visual mesh filename=../meshes/right_shoulder_roll_link.STL
- link right_shoulder_yaw_link: mass 0.082819 -> 0.0243504547323869; geometry collision mesh filename=../meshes/right_shoulder_yaw_link.STL; visual mesh filename=../meshes/right_shoulder_yaw_link.STL
- link right_wrist_yaw_link: mass 0.44922 -> 0.1244; geometry collision mesh filename=../meshes/right_wrist_yaw_link.STL; visual mesh filename=../meshes/right_wrist_yaw_link.STL
- link waist_yaw_link: mass 8.9679 -> 13.9790042253896; geometry collision box size=0.15 0.2 0.3; visual mesh filename=../meshes/waist_yaw_link.STL
Joints:
- removed joint auxiliary_left_leg_ankle_roll_joint1
- removed joint auxiliary_left_leg_ankle_roll_joint2
- removed joint auxiliary_left_leg_ankle_roll_joint3
- removed joint auxiliary_left_leg_ankle_roll_joint4
- removed joint auxiliary_right_leg_ankle_roll_joint1
- removed joint auxiliary_right_leg_ankle_roll_joint2
- removed joint auxiliary_right_leg_ankle_roll_joint3
- removed joint auxiliary_right_leg_ankle_roll_joint4
- removed joint keyframe_head_joint
- added joint left_hand_joint: type fixed, parent left_wrist_yaw_link, child left_hand_link, origin xyz=0 0 -0.1 rpy=0 0 0, axis 0 0 -1, limit lower=0 upper=0 effort=0 velocity=0
- added joint right_hand_joint: type fixed, parent right_wrist_yaw_link, child right_hand_link, origin xyz=0 0 -0.103 rpy=0 0 0, axis 0 0 1, limit lower=0 upper=0 effort=0 velocity=0
- joint head_pitch_joint: origin xyz=0 -0.026 0.046 rpy=0 0 0 -> xyz=0 0 0.046 rpy=0 0 0
- joint head_yaw_joint: origin xyz=0 0 0.37025 rpy=0 0 0 -> xyz=0 0 0.362300000000225 rpy=0 0 0
- joint left_elbow_pitch_joint: limit lower=-2.0944 upper=0 effort=65 velocity=26 -> lower=-1.8675 upper=0 effort=80 velocity=26; origin xyz=0 0 -0.06485 rpy=0 0 0 -> xyz=0 0 -0.0609999999999984 rpy=0 0 0
- joint left_leg_ankle_pitch_joint: limit lower=-0.87266 upper=0.50614 effort=70 velocity=14 -> lower=-0.87266 upper=0.50614 effort=100 velocity=14; origin xyz=0 0 -0.453 rpy=0 0 0 -> xyz=0 0 -0.453000000000091 rpy=0 0 0
- joint left_leg_ankle_roll_joint: limit lower=-0.50614 upper=0.50614 effort=70 velocity=14 -> lower=-0.50614 upper=0.50614 effort=100 velocity=14
- joint left_leg_knee_pitch_joint: limit lower=0 upper=2.5307 effort=250 velocity=14 -> lower=0 upper=2.5307 effort=200 velocity=14; origin xyz=-0.02 0 -0.2735 rpy=0 0 0 -> xyz=-0.0200000000000002 0 -0.273499999999999 rpy=0 0 0
- joint left_leg_pelvic_pitch_joint: limit lower=-1.9199 upper=1.5708 effort=250 velocity=14 -> lower=-1.9199 upper=1.5708 effort=200 velocity=14; origin xyz=0 0.061 -0.070239 rpy=0 0 0 -> xyz=0 0.061 0.0574999999999996 rpy=0 0 0
- joint left_leg_pelvic_roll_joint: limit lower=-0.17453 upper=1.5708 effort=150 velocity=14 -> lower=-0.17453 upper=1.5708 effort=200 velocity=14; origin xyz=-0.0028 0.0815 -0.055 rpy=0 0 0 -> xyz=-0.00280000000000061 0.0815 -0.0550000000000001 rpy=0 0 0
- joint left_leg_pelvic_yaw_joint: limit lower=-1.5708 upper=1.5708 effort=150 velocity=14 -> lower=-1.5708 upper=1.5708 effort=110 velocity=14; origin xyz=0 0 -0.0975 rpy=0 0 0 -> xyz=0 0 -0.0975000000000059 rpy=0 0 0
- joint left_shoulder_pitch_joint: limit lower=-3.1416 upper=1.0472 effort=65 velocity=26 -> lower=-3.1416 upper=1.0472 effort=80 velocity=26; origin xyz=0 0.1493 0.2753 rpy=0 0 -1.8248E-05 -> xyz=0 0.14500020317258 0.267300000000226 rpy=0 0 0
- joint left_shoulder_roll_joint: limit lower=-0.3491 upper=3.1416 effort=65 velocity=26 -> lower=-0.3491 upper=3.1416 effort=80 velocity=26; origin xyz=0 0.0536 0 rpy=0.1745 0 0 -> xyz=0 0.057 0 rpy=0.1745 0 0
- joint left_shoulder_yaw_joint: origin xyz=0.0001 0 -0.12765 rpy=0 0 0 -> xyz=0 0 -0.1315 rpy=0 0 0
- joint left_wrist_yaw_joint: origin xyz=0 0 -0.12165 rpy=0 0 0 -> xyz=0 0 -0.131 rpy=0 0 0; type revolute -> fixed
- joint right_elbow_pitch_joint: limit lower=-2.0944 upper=0 effort=65 velocity=26 -> lower=-1.8675 upper=0 effort=80 velocity=26; origin xyz=0 0 -0.06485 rpy=0 0 0 -> xyz=0 0 -0.0610000000000009 rpy=0 0 0
- joint right_leg_ankle_pitch_joint: limit lower=-0.87266 upper=0.50614 effort=70 velocity=14 -> lower=-0.87266 upper=0.50614 effort=100 velocity=14; origin xyz=0 0 -0.453 rpy=0 0 0 -> xyz=0 0 -0.45300000000003 rpy=0 0 0
- joint right_leg_ankle_roll_joint: limit lower=-0.50614 upper=0.50614 effort=70 velocity=14 -> lower=-0.50614 upper=0.50614 effort=100 velocity=14
- joint right_leg_knee_pitch_joint: limit lower=0 upper=2.5307 effort=250 velocity=14 -> lower=0 upper=2.5307 effort=200 velocity=14; origin xyz=-0.02 0 -0.2735 rpy=0 0 0 -> xyz=-0.0200000000000365 0 -0.273500000000063 rpy=0 0 0
- joint right_leg_pelvic_pitch_joint: limit lower=-1.9199 upper=1.5708 effort=250 velocity=14 -> lower=-1.9199 upper=1.5708 effort=200 velocity=14; origin xyz=0 -0.061 -0.070239 rpy=0 0 0 -> xyz=0 -0.0609999999999999 0.0575000000000002 rpy=0 0 0
- joint right_leg_pelvic_roll_joint: limit lower=-1.5708 upper=0.17453 effort=150 velocity=14 -> lower=-1.5708 upper=0.17453 effort=200 velocity=14; origin xyz=-0.0028 -0.0815 -0.055 rpy=0 0 0 -> xyz=-0.0028000000000013 -0.0814999999999976 -0.0549999999999963 rpy=0 0 0
- joint right_leg_pelvic_yaw_joint: limit lower=-1.5708 upper=1.5708 effort=150 velocity=14 -> lower=-1.5708 upper=1.5708 effort=110 velocity=14; origin xyz=0 0 -0.0975 rpy=0 0 0 -> xyz=0 0 -0.0975000000000075 rpy=0 0 0
- joint right_shoulder_pitch_joint: limit lower=-3.1416 upper=1.0472 effort=65 velocity=26 -> lower=-3.1416 upper=1.0472 effort=80 velocity=26; origin xyz=0 -0.1493 0.2753 rpy=0 0 0 -> xyz=0 -0.14499979682742 0.267300000000224 rpy=0 0 0
- joint right_shoulder_roll_joint: limit lower=-3.1416 upper=0.3491 effort=65 velocity=26 -> lower=-3.1416 upper=0.3491 effort=80 velocity=26; origin xyz=0 -0.0536 0 rpy=-0.1745 0 0 -> xyz=0 -0.057 0 rpy=-0.1745 0 0
- joint right_shoulder_yaw_joint: origin xyz=0.0001 0 -0.12765 rpy=0 0 0 -> xyz=0 0 -0.1315 rpy=0 0 0
- joint right_wrist_yaw_joint: origin xyz=0 0 -0.12165 rpy=0 0 0 -> xyz=0 0 -0.128 rpy=0 0 0; type revolute -> fixed
- joint waist_yaw_joint: axis 0 0 1 -> 0 0 -1; origin xyz=0 0 0.0185 rpy=0 0 0 -> xyz=0 0 0.154238635424338 rpy=0 0 0
