Commit message: 调小了P值和增大力矩限制

File: legged_gym/resources/robots/02/CASBOT_02.urdf (robot description, URDF)
Before this commit: robot CASBOT_02, 35 links, 34 joints
Joints:
- joint left_leg_knee_pitch_joint: limit lower=0 upper=2.5307 effort=150 velocity=14 -> lower=0 upper=2.5307 effort=250 velocity=14
- joint left_leg_pelvic_pitch_joint: limit lower=-1.9199 upper=1.5708 effort=150 velocity=14 -> lower=-1.9199 upper=1.5708 effort=250 velocity=14
- joint left_leg_pelvic_yaw_joint: limit lower=-1.5708 upper=1.5708 effort=60 velocity=14 -> lower=-1.5708 upper=1.5708 effort=150 velocity=14
- joint right_leg_knee_pitch_joint: limit lower=0 upper=2.5307 effort=150 velocity=14 -> lower=0 upper=2.5307 effort=250 velocity=14
- joint right_leg_pelvic_pitch_joint: limit lower=-1.9199 upper=1.5708 effort=150 velocity=14 -> lower=-1.9199 upper=1.5708 effort=250 velocity=14
- joint right_leg_pelvic_yaw_joint: limit lower=-1.5708 upper=1.5708 effort=60 velocity=14 -> lower=-1.5708 upper=1.5708 effort=150 velocity=14
- joint waist_yaw_joint: limit lower=-1.5708 upper=1.5708 effort=60 velocity=14 -> lower=-1.5708 upper=1.5708 effort=100 velocity=14

Commit message: Sim2sim works, but might have problem on the last dim in observation

File: legged_gym/resources/robots/02/CASBOT_02.urdf (robot description, URDF)
Before this commit: robot CASBOT_02, 35 links, 34 joints
Links:
- link left_shoulder_pitch_link: geometry visual mesh filename=meshes/left_shoulder_pitch_link.STL
- link right_shoulder_pitch_link: geometry visual mesh filename=meshes/right_shoulder_pitch_link.STL
Joints:
- joint left_leg_pelvic_yaw_joint: limit lower=-1.5708 upper=1.5708 effort=60 velocity=14 -> lower=-0.5 upper=1.5708 effort=60 velocity=14
- joint right_leg_pelvic_yaw_joint: limit lower=-1.5708 upper=1.5708 effort=60 velocity=14 -> lower=-1.5708 upper=0.5 effort=60 velocity=14

Commit message: update config_0627

File: legged_gym/resources/robots/02/CASBOT_02.urdf (robot description, URDF)
Before this commit: robot CASBOT_02, 35 links, 34 joints
Links:
- link left_shoulder_pitch_link: geometry collision mesh filename=meshes/left_shoulder_pitch_link.STL; visual mesh filename=meshes/left_shoulder_pitch_link.STL
- link right_shoulder_pitch_link: geometry collision mesh filename=meshes/right_shoulder_pitch_link.STL; visual mesh filename=meshes/right_shoulder_pitch_link.STL
Joints:
- joint left_leg_knee_pitch_joint: limit lower=0 upper=2.5307 effort=150 velocity=14 -> lower=0 upper=2.5307 effort=250 velocity=14
- joint left_leg_pelvic_pitch_joint: limit lower=-1.9199 upper=1.5708 effort=150 velocity=14 -> lower=-1.9199 upper=1.5708 effort=250 velocity=14
- joint left_leg_pelvic_roll_joint: limit lower=-0.17453 upper=1.5708 effort=150 velocity=14 -> lower=-0.17453 upper=1.5708 effort=120 velocity=14
- joint left_leg_pelvic_yaw_joint: limit lower=-0.5 upper=1.5708 effort=60 velocity=14 -> lower=-1.5708 upper=1.5708 effort=120 velocity=14
- joint right_leg_knee_pitch_joint: limit lower=0 upper=2.5307 effort=150 velocity=14 -> lower=0 upper=2.5307 effort=250 velocity=14
- joint right_leg_pelvic_pitch_joint: limit lower=-1.9199 upper=1.5708 effort=150 velocity=14 -> lower=-1.9199 upper=1.5708 effort=250 velocity=14
- joint right_leg_pelvic_roll_joint: limit lower=-1.5708 upper=0.17453 effort=150 velocity=14 -> lower=-1.5708 upper=0.17453 effort=120 velocity=14
- joint right_leg_pelvic_yaw_joint: limit lower=-1.5708 upper=0.5 effort=60 velocity=14 -> lower=-1.5708 upper=1.5708 effort=120 velocity=14
- joint waist_yaw_joint: limit lower=-1.5708 upper=1.5708 effort=60 velocity=14 -> lower=-1.5708 upper=1.5708 effort=120 velocity=14

Commit message: update config

File: legged_gym/resources/robots/02/CASBOT_02.urdf (robot description, URDF)
Before this commit: robot CASBOT_02, 35 links, 34 joints
Joints:
- joint left_leg_knee_pitch_joint: limit lower=0 upper=2.5307 effort=250 velocity=14 -> lower=0 upper=2.5307 effort=150 velocity=14
- joint left_leg_pelvic_pitch_joint: limit lower=-1.9199 upper=1.5708 effort=250 velocity=14 -> lower=-1.9199 upper=1.5708 effort=150 velocity=14
- joint left_leg_pelvic_roll_joint: limit lower=-0.17453 upper=1.5708 effort=120 velocity=14 -> lower=-0.17453 upper=1.5708 effort=150 velocity=14
- joint left_leg_pelvic_yaw_joint: limit lower=-1.5708 upper=1.5708 effort=120 velocity=14 -> lower=-1.5708 upper=1.5708 effort=60 velocity=14
- joint right_leg_knee_pitch_joint: limit lower=0 upper=2.5307 effort=250 velocity=14 -> lower=0 upper=2.5307 effort=150 velocity=14
- joint right_leg_pelvic_pitch_joint: limit lower=-1.9199 upper=1.5708 effort=250 velocity=14 -> lower=-1.9199 upper=1.5708 effort=150 velocity=14
- joint right_leg_pelvic_roll_joint: limit lower=-1.5708 upper=0.17453 effort=120 velocity=14 -> lower=-1.5708 upper=0.17453 effort=150 velocity=14
- joint right_leg_pelvic_yaw_joint: limit lower=-1.5708 upper=1.5708 effort=120 velocity=14 -> lower=-1.5708 upper=1.5708 effort=60 velocity=14
- joint waist_yaw_joint: limit lower=-1.5708 upper=1.5708 effort=120 velocity=14 -> lower=-1.5708 upper=1.5708 effort=60 velocity=14

Commit message: 存一版

File: legged_gym/resources/robots/02/CASBOT_02.urdf (robot description, URDF)
Before this commit: robot CASBOT_02, 35 links, 34 joints
Joints:
- joint left_leg_pelvic_yaw_joint: limit lower=-0.5 upper=1.5708 effort=150 velocity=14 -> lower=-1.5708 upper=1.5708 effort=150 velocity=14
- joint right_leg_pelvic_yaw_joint: limit lower=-1.5708 upper=0.5 effort=60 velocity=14 -> lower=-1.5708 upper=1.5708 effort=150 velocity=14

Commit message: 稳定站立版本,mujoco里有点抖

File: legged_gym/resources/robots/02/CASBOT_02.urdf (robot description, URDF)
Before this commit: robot CASBOT_02, 35 links, 34 joints
Joints:
- joint left_leg_ankle_pitch_joint: limit lower=-0.87266 upper=0.50614 effort=60 velocity=14 -> lower=-0.87266 upper=0.50614 effort=70 velocity=14
- joint left_leg_ankle_roll_joint: limit lower=-0.50614 upper=0.50614 effort=60 velocity=14 -> lower=-0.50614 upper=0.50614 effort=70 velocity=14
- joint right_leg_ankle_pitch_joint: limit lower=-0.87266 upper=0.50614 effort=60 velocity=14 -> lower=-0.87266 upper=0.50614 effort=70 velocity=14
- joint right_leg_ankle_roll_joint: limit lower=-0.50614 upper=0.50614 effort=60 velocity=14 -> lower=-0.50614 upper=0.50614 effort=70 velocity=14

Commit message: update new reward

File: legged_gym/resources/robots/02/CASBOT_02.urdf (robot description, URDF)
Before this commit: robot CASBOT_02, 35 links, 34 joints
Joints:
- joint head_pitch_joint: limit lower=-0.2618 upper=0.5236 effort=60 velocity=14 -> lower=-0.2618 upper=0.5236 effort=65 velocity=14
- joint head_yaw_joint: limit lower=-1.5708 upper=1.5708 effort=60 velocity=14 -> lower=-1.5708 upper=1.5708 effort=65 velocity=14
- joint left_leg_ankle_pitch_joint: limit lower=-0.87266 upper=0.50614 effort=60 velocity=14 -> lower=-0.87266 upper=0.50614 effort=70 velocity=14
- joint left_leg_ankle_roll_joint: limit lower=-0.50614 upper=0.50614 effort=60 velocity=14 -> lower=-0.50614 upper=0.50614 effort=70 velocity=14
- joint left_leg_pelvic_yaw_joint: limit lower=-1.5708 upper=1.5708 effort=60 velocity=14 -> lower=-1.5708 upper=1.5708 effort=70 velocity=14
- joint right_leg_ankle_pitch_joint: limit lower=-0.87266 upper=0.50614 effort=60 velocity=14 -> lower=-0.87266 upper=0.50614 effort=70 velocity=14
- joint right_leg_ankle_roll_joint: limit lower=-0.50614 upper=0.50614 effort=60 velocity=14 -> lower=-0.50614 upper=0.50614 effort=70 velocity=14
- joint right_leg_pelvic_yaw_joint: limit lower=-1.5708 upper=1.5708 effort=60 velocity=14 -> lower=-1.5708 upper=1.5708 effort=70 velocity=14
- joint waist_yaw_joint: limit lower=-1.5708 upper=1.5708 effort=60 velocity=14 -> lower=-1.5708 upper=1.5708 effort=70 velocity=14

Commit message: jiamoxing

File: legged_gym/resources/robots/02/CASBOT_02.urdf (robot description, URDF)
Before this commit: robot CASBOT_02, 35 links, 34 joints
Links:
- link base_link: geometry visual mesh filename=/home/casbot/ZHZ_ws/HoST/legged_gym/resources/robots/02/mes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
- link head_pitch_link: geometry collision mesh filename=/home/casbot/ZHZ_ws/HoST/legged_gym/resources/robots/02/mes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; visual mesh filename=/home/casbot/ZHZ_ws/HoST/legged_gym/resources/robots/02/mes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
- link head_yaw_link: geometry collision mesh filename=/home/casbot/ZHZ_ws/HoST/legged_gym/resources/robots/02/mes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; visual mesh filename=/home/casbot/ZHZ_ws/HoST/legged_gym/resources/robots/02/mes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
- link left_elbow_pitch_link: geometry collision mesh filename=/home/casbot/ZHZ_ws/HoST/legged_gym/resources/robots/02/mes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; visual mesh filename=/home/casbot/ZHZ_ws/HoST/legged_gym/resources/robots/02/mes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
- link left_leg_ankle_pitch_link: geometry visual mesh filename=/home/casbot/ZHZ_ws/HoST/legged_gym/resources/robots/02/mes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
- link left_leg_ankle_roll_link: geometry collision sphere radius=0.005; collision sphere radius=0.005
- link left_leg_knee_pitch_link: geometry collision box size=0.03 0.06 0.1; collision box size=0.05 0.07 0.19
- link left_leg_pelvic_pitch_link: geometry collision mesh filename=/home/casbot/ZHZ_ws/HoST/legged_gym/resources/robots/02/mes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; visual mesh filename=/home/casbot/ZHZ_ws/HoST/legged_gym/resources/robots/02/mes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
- link left_leg_pelvic_roll_link: geometry collision mesh filename=/home/casbot/ZHZ_ws/HoST/legged_gym/resources/robots/02/mes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; visual mesh filename=/home/casbot/ZHZ_ws/HoST/legged_gym/resources/robots/02/mes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
- link left_leg_pelvic_yaw_link: geometry collision mesh filename=/home/casbot/ZHZ_ws/HoST/legged_gym/resources/robots/02/mes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; visual mesh filename=/home/casbot/ZHZ_ws/HoST/legged_gym/resources/robots/02/mes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
- link left_shoulder_pitch_link: geometry visual mesh filename=/home/casbot/ZHZ_ws/HoST/legged_gym/resources/robots/02/mes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
- link left_shoulder_roll_link: geometry collision mesh filename=/home/casbot/ZHZ_ws/HoST/legged_gym/resources/robots/02/mes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; visual mesh filename=/home/casbot/ZHZ_ws/HoST/legged_gym/resources/robots/02/mes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
- link left_shoulder_yaw_link: geometry collision mesh filename=/home/casbot/ZHZ_ws/HoST/legged_gym/resources/robots/02/mes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; visual mesh filename=/home/casbot/ZHZ_ws/HoST/legged_gym/resources/robots/02/mes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
- link left_wrist_yaw_link: geometry collision mesh filename=/home/casbot/ZHZ_ws/HoST/legged_gym/resources/robots/02/mes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; visual mesh filename=/home/casbot/ZHZ_ws/HoST/legged_gym/resources/robots/02/mes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
- link right_elbow_pitch_link: geometry collision mesh filename=/home/casbot/ZHZ_ws/HoST/legged_gym/resources/robots/02/mes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; visual mesh filename=/home/casbot/ZHZ_ws/HoST/legged_gym/resources/robots/02/mes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
- link right_leg_ankle_pitch_link: geometry visual mesh filename=/home/casbot/ZHZ_ws/HoST/legged_gym/resources/robots/02/mes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
- link right_leg_ankle_roll_link: geometry collision sphere radius=0.005; collision sphere radius=0.005
- link right_leg_knee_pitch_link: geometry collision box size=0.03 0.06 0.1; collision box size=0.05 0.07 0.19
- link right_leg_pelvic_pitch_link: geometry collision mesh filename=/home/casbot/ZHZ_ws/HoST/legged_gym/resources/robots/02/mes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; visual mesh filename=/home/casbot/ZHZ_ws/HoST/legged_gym/resources/robots/02/mes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
- link right_leg_pelvic_roll_link: geometry collision mesh filename=/home/casbot/ZHZ_ws/HoST/legged_gym/resources/robots/02/mes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; visual mesh filename=/home/casbot/ZHZ_ws/HoST/legged_gym/resources/robots/02/mes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
- link right_leg_pelvic_yaw_link: geometry collision mesh filename=/home/casbot/ZHZ_ws/HoST/legged_gym/resources/robots/02/mes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; visual mesh filename=/home/casbot/ZHZ_ws/HoST/legged_gym/resources/robots/02/mes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
- link right_shoulder_pitch_link: geometry visual mesh filename=/home/casbot/ZHZ_ws/HoST/legged_gym/resources/robots/02/mes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
- link right_shoulder_roll_link: geometry collision mesh filename=/home/casbot/ZHZ_ws/HoST/legged_gym/resources/robots/02/mes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; visual mesh filename=/home/casbot/ZHZ_ws/HoST/legged_gym/resources/robots/02/mes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
- link right_shoulder_yaw_link: geometry collision mesh filename=/home/casbot/ZHZ_ws/HoST/legged_gym/resources/robots/02/mes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; visual mesh filename=/home/casbot/ZHZ_ws/HoST/legged_gym/resources/robots/02/mes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
- link right_wrist_yaw_link: geometry collision mesh filename=/home/casbot/ZHZ_ws/HoST/legged_gym/resources/robots/02/mes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; visual mesh filename=/home/casbot/ZHZ_ws/HoST/legged_gym/resources/robots/02/mes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
- link waist_yaw_link: geometry collision mesh filename=/home/casbot/ZHZ_ws/HoST/legged_gym/resources/robots/02/mes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; visual mesh filename=/home/casbot/ZHZ_ws/HoST/legged_gym/resources/robots/02/mes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
Joints:
- joint left_leg_pelvic_pitch_joint: limit lower=-1.9199 upper=1.5708 effort=250 velocity=14 -> lower=-1.9199 upper=1.5708 effort=200 velocity=14
- joint left_leg_pelvic_roll_joint: limit lower=-0.17453 upper=1.5708 effort=150 velocity=14 -> lower=-0.17453 upper=1.5708 effort=200 velocity=14
- joint left_leg_pelvic_yaw_joint: limit lower=-1.5708 upper=1.5708 effort=150 velocity=14 -> lower=-1.5708 upper=1.5708 effort=100 velocity=14
- joint right_leg_pelvic_pitch_joint: limit lower=-1.9199 upper=1.5708 effort=250 velocity=14 -> lower=-1.9199 upper=1.5708 effort=200 velocity=14
- joint right_leg_pelvic_roll_joint: limit lower=-1.5708 upper=0.17453 effort=150 velocity=14 -> lower=-1.5708 upper=0.17453 effort=200 velocity=14
- joint right_leg_pelvic_yaw_joint: limit lower=-1.5708 upper=1.5708 effort=150 velocity=14 -> lower=-1.5708 upper=1.5708 effort=100 velocity=14

Commit message: dunqi

File: legged_gym/resources/robots/02/CASBOT_02.urdf (robot description, URDF)
Before this commit: robot CASBOT_02, 35 links, 34 joints
Joints:
- joint left_shoulder_pitch_joint: limit lower=-3.1416 upper=1.0472 effort=65 velocity=26 -> lower=-1.5716 upper=1.0472 effort=65 velocity=26
- joint left_shoulder_roll_joint: limit lower=-0.3491 upper=3.1416 effort=65 velocity=26 -> lower=-0.0 upper=1.5716 effort=65 velocity=26
- joint right_shoulder_pitch_joint: limit lower=-3.1416 upper=1.0472 effort=65 velocity=26 -> lower=-1.5716 upper=1.0472 effort=65 velocity=26
- joint right_shoulder_roll_joint: limit lower=-3.1416 upper=0.3491 effort=65 velocity=26 -> lower=-1.5716 upper=0.0 effort=65 velocity=26
