Commit message: save for update

File: legged_gym/resources/robots/02/CASBOT_02.urdf (robot description, URDF)
Before this commit: robot CASBOT_02, 35 links, 34 joints
Joints:
- joint left_leg_pelvic_yaw_joint: limit lower=-0.5 upper=1.5708 effort=60 velocity=14 -> lower=-1.5708 upper=1.5708 effort=60 velocity=14
